Commit message: creating r2d2 robot with URDF and setting up controls to be used with turtle_teleop_key node. 01/04/2023

File: src/mark_r2d2/urdf/r2d2.urdf.xacro (robot description, xacro)
@@ -1,4 +1,5 @@
 <?xml version="1.0"?>
 <robot name="macroed_r2d2" xmlns:xacro="http://ros.org/wiki/xacro">
+<!-- This is a comment in the XML file -->
   <xacro:property name="width" value="0.2" />
   <xacro:property name="leglen" value="0.6" />
@@ -25,4 +26,5 @@
   <link name="base_link">
     <visual>
+      <origin xyz="0 0 0" rpy="0 0 0" />
       <geometry>
         <cylinder radius="${width}" length="${bodylen}"/>
@@ -31,4 +33,5 @@
     </visual>
     <collision>
+      <origin xyz="0 0 0" rpy="0 0 0" />
       <geometry>
         <cylinder radius="${width}" length="${bodylen}"/>
@@ -214,3 +217,30 @@
     <origin xyz="${.707*width+0.04} 0 ${.707*width}"/>
   </joint>
+ <link name="eye">
+    <visual>
+      <geometry>
+       <cylinder radius="0.02" length="0.02"/>
+      </geometry>
+      <material name="black"/>
+      <origin rpy="0 1.57075 0" xyz="0 0 0"/>
+    </visual>
+    <collision>
+      <geometry>
+        <cylinder radius="0.02" length="0.02"/>
+      </geometry>
+      <origin rpy="0 1.57075 0" xyz="0 0 0"/>
+    </collision>
+    <xacro:default_inertial mass="1"/>
+  </link>
+  <joint name="socket" type="fixed">
+    <parent link="box"/>
+    <child link="eye"/>
+    <origin xyz="0 0 0"/>
+ </joint>
+  <link name="base_footprint"/>
+  <joint name="base_footprint_to_base_link" type="fixed">
+    <parent link="base_footprint"/>
+    <child link="base_link"/>
+    <origin xyz="0 0 ${-0.25+leglen+wheeldiam/2+.05+wheeldiam/2}" />
+  </joint>
 </robot>

Commit message: Commit of assingment 3, r2d2 is moving, collision is clunky with some errors.

File: src/mark_r2d2/urdf/r2d2.urdf.xacro (robot description, xacro)
@@ -2,4 +2,5 @@
 <robot name="macroed_r2d2" xmlns:xacro="http://ros.org/wiki/xacro">
 <!-- This is a comment in the XML file -->
+  <xacro:arg name="laser_visual" default="false"/>
   <xacro:property name="width" value="0.2" />
   <xacro:property name="leglen" value="0.6" />
@@ -244,3 +245,81 @@
     <origin xyz="0 0 ${-0.25+leglen+wheeldiam/2+.05+wheeldiam/2}" />
   </joint>
+  <joint name="scan_joint" type="fixed">
+    <parent link="eye"/>
+    <child link="base_scan"/>
+    <origin xyz="-0.02 0 0.06" rpy="0 0 0"/>
+  </joint>
+  <link name="base_scan">
+    <visual>
+      <origin xyz="0 0 0" rpy="0 0 0"/>
+      <geometry>
+        <mesh filename="package://turtlebot3_description/meshes/sensors/lds.stl" scale="0.001 0.001 0.001"/>
+      </geometry>
+      <material name="black"/>
+    </visual>
+    <collision>
+      <origin xyz="0 0 0" rpy="0 0 0"/>
+      <geometry>
+        <cylinder length="0.0315" radius="0.055"/>
+      </geometry>
+    </collision>
+    <inertial>
+      <mass value="0.114" />
+      <origin xyz="0 0 0" />
+      <inertia ixx="0.001" ixy="0.0" ixz="0.0"
+               iyy="0.001" iyz="0.0"
+               izz="0.001" />
+    </inertial>
+  </link>
+  <gazebo reference="base_scan">
+    <material>Gazebo/FlatBlack</material>
+    <sensor type="ray" name="lds_lfcd_sensor">
+      <pose>0 0 0 0 0 0</pose>
+      <visualize>$(arg laser_visual)</visualize>
+      <update_rate>5</update_rate>
+      <ray>
+        <scan>
+          <horizontal>
+            <samples>360</samples>
+            <resolution>1</resolution>
+            <min_angle>0.0</min_angle>
+            <max_angle>6.28319</max_angle>
+          </horizontal>
+        </scan>
+        <range>
+          <min>0.120</min>
+          <max>3.5</max>
+          <resolution>0.015</resolution>
+        </range>
+        <noise>
+          <type>gaussian</type>
+          <mean>0.0</mean>
+          <stddev>0.01</stddev>
+        </noise>
+      </ray>
+      <plugin name="gazebo_ros_lds_lfcd_controller" filename="libgazebo_ros_laser.so">
+        <topicName>scan</topicName>
+        <frameName>base_scan</frameName>
+      </plugin>
+    </sensor>
+  </gazebo>
+  <gazebo>
+<!-- Gazebo plugin for skid steering -->
+  <plugin name="skid_steer_drive_controller" filename="libgazebo_ros_skid_steer_drive.so">
+    <alwaysOn>true</alwaysOn>
+    <updateRate>50.0</updateRate>
+    <leftFrontJoint>left_front_wheel_joint</leftFrontJoint>
+    <rightFrontJoint>right_front_wheel_joint</rightFrontJoint>
+    <leftRearJoint>left_back_wheel_joint</leftRearJoint>
+    <rightRearJoint>right_back_wheel_joint</rightRearJoint>
+    <wheelSeparation>${2.0*baselen/3.0}</wheelSeparation>
+    <wheelDiameter>${wheeldiam}</wheelDiameter>
+	<torque>10</torque>
+	<broadcastTF>1</broadcastTF>
+	<odometryFrame>odom</odometryFrame>
+	<commandTopic>cmd_vel</commandTopic>
+	<odometryTopic>/odom</odometryTopic>
+	<robotBaseFrame>base_link</robotBaseFrame>
+  </plugin>
+</gazebo>
 </robot>

Commit message: Assignment 3, custom gazebo and gmapping

File: src/mark_r2d2/urdf/r2d2.urdf.xacro (robot description, xacro)
@@ -197,4 +197,5 @@
     <axis xyz="0 0 1"/>
     <origin xyz="0 0 ${bodylen/2}"/>
+    <dynamics damping="0.0" friction="0.9"/>
   </joint>
   <link name="box">
@@ -265,9 +266,5 @@
     </collision>
     <inertial>
-      <mass value="0.114" />
-      <origin xyz="0 0 0" />
-      <inertia ixx="0.001" ixy="0.0" ixz="0.0"
-               iyy="0.001" iyz="0.0"
-               izz="0.001" />
+	<xacro:default_inertial mass="0.1"/>
     </inertial>
   </link>

Commit message: little fixes to assignment 3

File: src/mark_r2d2/urdf/r2d2.urdf.xacro (robot description, xacro)
@@ -265,7 +265,5 @@
       </geometry>
     </collision>
-    <inertial>
-	<xacro:default_inertial mass="0.1"/>
-    </inertial>
+    <xacro:default_inertial mass="0.1"/>
   </link>
   <gazebo reference="base_scan">
